File: Focus_V8.brd (EAGLE design)
At the start: 64.8 x 94 mm, 100 parts, among them X1 USB+SHIELD, Y1 16Mhz

Commit message: Version 8 removes the Linear Light Array and uses a TSL1401CL-Adapter Board via a 5 pin JST SH connector. There is also a 3 pin JST connector for communicating with a Serial Enabled LCD display RGB LED has also been added to give a status indication.
Parts:
- removed +10V, -5V: PTR1TP20R, testpad:TP20R
- removed 7660: ICL7660CSA, maxim:SO08
- removed AD5531: AD5531BRUZ, BIG:RU_16
- removed C33: 10uF (1 Ohm ESR), SparkFun:EIA3216-KIT
- removed C35: 0.1uF, SparkFun:0603-CAP
- removed D2, D3: NXP - 1PS76SB21,115, SparkFun:SOD-323
- removed L: YELLOW, BIG:CHIPLED_0805
- added +12V, -12V: PTR1TP20R, testpad:TP20R
- added COM-07844: LED-TRICOLOR, SparkFun-LED:LED-TRICOLOR-SMD
- added IO11: M01SMD-4.5X1.5, SparkFun-Connectors:PAD-1.5X4.5
- added L3: 47uH, BIG:11R473C
- added LCD: LCD-09394, SparkFun-Connectors:JST-3-PTH
- added MEA1D0512SC: +12V/-12V, dc-dc-converter:NMA
- added R22, R23: 100, SparkFun:0603-RES
- added R24: 200, SparkFun:0603-RES
- added SENSOR: PRT-10209, SparkFun-Connectors:1X05-1MM-RA
- added SJ2: SOLDERJUMPERNO, SparkFun-Passives:SJ_2S-NO
- added U$2: (no value), BIG:SMD-22
- C10, C26, C34: value 0.1uF -> 1uF
- C30: value 10uF (1 Ohm ESR) -> 1uF; device SparkFun:EIA3216-KIT -> SparkFun:0603-CAP
- ON: value ON -> APA2106MGC
- R12, R15: value 10K -> 10K 0.1%
- R18: value 1K -> 200
- R5: value 300 -> 100
- RX, TX: value YELLOW -> APA2106SYCK
- U$1: value TSL1401CL -> AD5331; device BIG:TSL1401CL -> BIG:AD5531
- moved C30 20.7 mm to (41.5, 48.5)
- moved U$1 16.6 mm to (62.3, 48.9), turned to 180 degrees
- moved R18 15.2 mm to (54.6, 59.7)
- moved C39 13.6 mm to (50.8, 26.2), turned to 180 degrees
- moved C38 9.86 mm to (50.8, 22.4), turned to 180 degrees
- moved C24 9.67 mm to (52.6, 12.4)
- moved C25 9.57 mm to (56.4, 12.4)
- moved C26 9.54 mm to (48.3, 16.6)
- moved JP1 6.97 mm to (92.5, 2.54)
- moved C10 1.96 mm to (45.1, 38.4), turned to 180 degrees
- moved C42 1.91 mm to (56.1, 41.9)
- moved C43 1.91 mm to (56.1, 44.5)
- moved R5 1.91 mm to (65.4, 39.4)
- moved R2 0.64 mm to (56.3, 58.7)
- moved C34 0.36 mm to (40.6, 31.5), turned to 0 degrees
- renumbered Y1 to 16MHZ
Connections:
- net AD5531 renamed BNCVIN
- removed net +10V: +10V.TP, AD5531.16, AD8221.8, ADTL082-IC1.8, ADTL082-IC2.8, C16.1, C17.1, C24.A, C25.A, C26.2, C27.2, C28.2, C40.2, C41.2, C7.2, C8.2, D2.1
- removed net -5V: -5V.TP, 7660.5, AD5531.13, AD8221.5, ADTL082-IC1.4, ADTL082-IC2.4, C12.2, C13.2, C14.1, C15.1, C36.2, C37.2, C38.C, C39.C, C42.2, C43.2
- removed net N$27: L.ANODE, R18.1
- removed net TSL1401R_A0: ATMEGA32U4.28, U$1.AO
- new net +12V: +12V.TP, AD8221.8, ADTL082-IC1.8, ADTL082-IC2.8, C16.1, C17.1, C24.A, C25.A, C26.1, C27.2, C28.2, C40.2, C41.2, C7.2, C8.2, L3.P$2, U$1.VDD
- new net -12V: -12V.TP, AD8221.5, ADTL082-IC1.4, ADTL082-IC2.4, C12.2, C13.2, C14.1, C15.1, C26.2, C36.2, C37.2, C38.C, C39.C, C42.2, C43.2, MEA1D0512SC.4, U$1.VSS
- new net A0: ATMEGA32U4.36, R23.1
- new net AGND: AD7894-10.3, AD8221.6, BNCFOCUS1.GND, C12.1, C13.1, C14.2, C15.2, C16.2, C17.2, C19.1, C20.2, C21.2, C23.2, C24.C, C25.C, C27.1, C28.1, C31.2, C32.2, C36.1, C37.1, C38.A, C39.A, C4.2, C40.1, C41.1, C42.1, C43.1, C7.1, C8.1, MEA1D0512SC.5, R10.1, R17.1, R8.1, SJ2.1, U$1.DUTGND, U$1.GND
- new net IO12: ATMEGA32U4.26, R22.1
- new net N$29: COM-07844.R, R18.2
- new net N$6: L3.P$1, MEA1D0512SC.6
- new net TSL1401R_AO: ATMEGA32U4.30, SENSOR.4
- net +5V: now also C30.1, COM-07844.A, LCD.1, MEA1D0512SC.1, SENSOR.5; no longer 7660.8, D3.2, R18.2, U$1.VDD
- net 2.5V_REFIN: now also U$1.REFIN; no longer AD5531.2
- net D7: now also LCD.3
- net DAC_CLR: now also U$1.CLR; no longer AD5531.9
- net DAC_PD: now also U$1.PD; no longer AD5531.10
- net DAC_SS: now also U$1.SYNC; no longer AD5531.5
- net GND: now also C30.2, LCD.2, MEA1D0512SC.2, SENSOR.1, SJ2.2, U$1.LDAC, U$1.REFAGND, U$1.SDO; no longer 7660.3, AD5531.1, AD5531.11, AD5531.14, AD5531.3, AD5531.8, AD7894-10.3, AD8221.6, BNCFOCUS1.GND, C12.1, C13.1, C14.2, C15.2, C16.2, C17.2, C19.1, C20.2, C21.2, C23.2, C24.C, C25.C, C26.1, C27.1, C28.1, C31.2, C32.2, C35.1, C36.1, C37.1, C38.A, C39.A, C4.2, C40.1, C41.1, C42.1, C43.1, C7.1, C8.1, R10.1, R17.1, R8.1, U$1.GND1, U$1.GND2
- net IO13: now also R18.1; no longer L.CATHODE
- net MOSI: now also U$1.SDIN; no longer AD5531.4
- net N$28: now also ATMEGA32U4.12, IO11.P$1; no longer C30.A, D2.2, D3.1
- net N$3: now also R24.2; no longer R5.2
- net N$30: now also COM-07844.B, R22.2; no longer 7660.4, C33.C
- net N$31: now also COM-07844.G, R23.2; no longer 7660.2, C30.C, C33.A
- net N$5: now also R24.1, R5.2; no longer 7660.7, C35.2
- net N$8: now also U$1.VOUT; no longer AD5531.15
- net SCK: now also U$1.SCLK; no longer AD5531.7
- net TSL1401R_CLK: now also ATMEGA32U4.29, SENSOR.3; no longer ATMEGA32U4.30, U$1.CLK
- net TSL1401R_SI: now also ATMEGA32U4.28, SENSOR.2; no longer ATMEGA32U4.29, U$1.SI
Routing:
- net +12V: track 0.00 -> 154.0 mm, vias 0 -> 2
- net -5V: track 119.2 -> 0.00 mm, vias 3 -> 0
- net -12V: track 0.00 -> 115.6 mm, vias 0 -> 2
- net +10V: track 90.1 -> 0.00 mm, vias 5 -> 0
- net TSL1401R_A0: track 32.6 -> 0.00 mm
- net IO12: track 0.00 -> 32.1 mm, vias 0 -> 2
- net TSL1401R_AO: track 0.00 -> 31.7 mm
- net GND: track 58.4 -> 78.5 mm, vias 22 -> 15
- net IO13: track 23.3 -> 3.69 mm, vias 2 -> 0
- net AGND: track 0.00 -> 10.8 mm, vias 0 -> 10
- net D7: track 28.8 -> 38.7 mm
- net A0: track 0.00 -> 8.20 mm
- net TSL1401R_SI: track 23.5 -> 31.6 mm
- net N$6: track 0.00 -> 7.29 mm
- net N$28: track 7.13 -> 1.49 mm
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- added copper zone on layer 1, net AGND
- added copper zone on layer 16, net AGND
Other:
- board text added: "+12V/-12V Power Supply"
- board text added: "+5V"
- board text added: "AO"
- board text added: "CLK"
- board text added: "IO11"
- board text added: "IO12"
- board text added: "RX"
- board text added: "SI"
- board text removed: "+10V/-5V Power Supply"
- board text removed: "Caps C24,C25,C38,C39 might not need to be low ESR"
- board text removed: "Optional Cap (C35)"
- board text removed: "slows the OSC (pin 7)"
